Commit message: included camera sensor

File: src/rosbot_description/urdf/rosbot.xacro (robot description, xacro)
@@ -85,4 +85,31 @@
   </collision>
 </link>
+<!-- ========== CAMERA LINK ADDED ========== -->
+<link name="camera_link">
+  <inertial>
+    <origin xyz="0 0 0" rpy="0 0 0"/>
+    <mass value="0.05"/>
+    <inertia ixx="0.0001" iyy="0.0001" izz="0.0001" ixy="0" iyz="0" ixz="0"/>
+  </inertial>
+  <visual>
+    <origin xyz="0.02 0 0" rpy="0 0 0"/>
+    <geometry>
+      <box size="0.03 0.03 0.03"/>
+    </geometry>
+    <material name="black"/>
+  </visual>
+  <collision>
+    <origin xyz="0.06 0 0.10" rpy="0 0 0"/>
+    <geometry>
+      <box size="0.03 0.03 0.03"/>
+    </geometry>
+  </collision>
+</link>
+<!-- ========== CAMERA JOINT ADDED ========== -->
+<joint name="camera_joint" type="fixed">
+  <origin xyz="0.08 0.0 0.18" rpy="0 0 0"/>
+  <parent link="base_link"/>
+  <child link="camera_link"/>
+</joint>
 <joint name="base_joint" type="fixed">
   <origin xyz="0.0 0.0 0.0" rpy="0 0 0"/>
