Commit message: modified xacro files

File: src/rosbot_description/urdf/materials.xacro (robot description, xacro)
@@ -1,12 +1,12 @@
 <?xml version="1.0" ?>
 <robot name="rosbot" xmlns:xacro="http://www.ros.org/wiki/xacro" >
-<material name="orange">
-  <color rgba="1.0 0.4235 0.0392 1"/>
+<material name="silver">
+  <color rgba="0.700 0.700 0.700 1.000"/>
 </material>
 <material name="black">
-  <color rgba="0 0 0 1"/>
+  <color rgba="0 0 0 1.000"/>
 </material>
-<material name="grey">
-  <color rgba="0.5 0.5 0.5 1"/>
+<material name="orange">
+  <color rgba="1.0 0.5 0.5 1.000"/>
 </material>
 </robot>

File: src/rosbot_description/urdf/rosbot.xacro (robot description, xacro)
@@ -36,5 +36,5 @@
       <mesh filename="file://$(find rosbot_description)/meshes/right_wheel_1.stl" scale="0.001 0.001 0.001"/>
     </geometry>
-    <material name="grey"/>
+    <material name="silver"/>
   </visual>
   <collision>
@@ -56,5 +56,5 @@
       <mesh filename="file://$(find rosbot_description)/meshes/left_wheel_1.stl" scale="0.001 0.001 0.001"/>
     </geometry>
-    <material name="grey"/>
+    <material name="silver"/>
   </visual>
   <collision>
@@ -85,31 +85,4 @@
   </collision>
 </link>
-<!-- ========== CAMERA LINK ADDED ========== -->
-<link name="camera_link">
-  <inertial>
-    <origin xyz="0 0 0" rpy="0 0 0"/>
-    <mass value="0.05"/>
-    <inertia ixx="0.0001" iyy="0.0001" izz="0.0001" ixy="0" iyz="0" ixz="0"/>
-  </inertial>
-  <visual>
-    <origin xyz="0.02 0 0" rpy="0 0 0"/>
-    <geometry>
-      <box size="0.03 0.03 0.03"/>
-    </geometry>
-    <material name="black"/>
-  </visual>
-  <collision>
-    <origin xyz="0.06 0 0.10" rpy="0 0 0"/>
-    <geometry>
-      <box size="0.03 0.03 0.03"/>
-    </geometry>
-  </collision>
-</link>
-<!-- ========== CAMERA JOINT ADDED ========== -->
-<joint name="camera_joint" type="fixed">
-  <origin xyz="0.08 0.0 0.18" rpy="0 0 0"/>
-  <parent link="base_link"/>
-  <child link="camera_link"/>
-</joint>
 <joint name="base_joint" type="fixed">
   <origin xyz="0.0 0.0 0.0" rpy="0 0 0"/>
